File: Alpenglow_FUterus_PCB.kicad_pcb (KiCad board)
At the start: 2 copper layers, 76.2 x 76.2 mm, 16 parts, among them SW1 SW_SLIDE

Commit message: Re-made Squiggles component, removed extras from PCB, fixed center LED+ squiggle so it's not close to GND pads
Parts:
- removed the ? at (178.4, 30.8)
- removed the ? at (207.0, 111.7)
- removed the ? at (205.2, 99.2)
- removed the ? at (199.3, 76.9)
- removed the ? at (242.0, 85.2)

Commit message: silk component text tweaks
Parts:
- removed the ? at (167.0, 107.4)
- added ?: , clipboard:9932db26-c585-4969-88a4-3276315666fc, F.Cu at (125.5, 104.9)
- added ?: , clipboard:978c0960-0638-40cb-9598-f7584c1d72e6, F.Cu at (163.1, 93.6)
- D1, D2, D3: footprint LED_THT:LED_D5.0mm_Horizontal_O3.81mm_Z3.0mm -> Alpenglow:LED_D5.0mm_Horizontal_O3.81mm_Z3.0mm_copy
