File: Alpenglow_FUterus_PCB.kicad_pcb (KiCad board)
At the start: 2 copper layers, 76.2 x 76.2 mm, 12 parts, among them SW1 SW_SLIDE

Commit message: updated battery holder for text fields
Parts:
- D1, D2, D3: footprint Alpenglow:LED_D5.0mm_Horizontal_O3.81mm_Z3.0mm_copy -> Alpenglow:LED_D5.0mm_Horizontal
Changed lines of the file:
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@@
+			)
+		)
+		(property "Plus" "+"
+			(at 8.675619 -0.337093 55)
+			(layer "B.SilkS")
+			(effects
+				(font
+					(size 2 2)
+					(thickness 0.15)
+				)
+				(justify mirror)
+			)
+		)
+		(property "Minus" "-"
+			(at -3.4 0.2 55)
+			(layer "B.SilkS")
+			(effects
+				(font
+					(size 2 2)
+					(thickness 0.15)
+				)
+				(justify mirror)
 			)
 		)
@@
 			(layer "B.SilkS")
 		)
-		(fp_text user "+"
-			(at 9.000001 0.05 55)
+		(fp_text user "${REFERENCE}"
+			(at -6 13 0)
 			(unlocked yes)
 			(layer "B.SilkS")
 			(effects
 				(font
-					(size 2 2)
-					(thickness 0.15)
-				)
-				(justify mirror)
-			)
-		)
-		(fp_text user "${REFERENCE}"
-			(at 11.074868 -8.243016 0)
-			(unlocked yes)
-			(layer "B.SilkS")
-			(effects
-				(font
 					(size 1 1)
 					(thickness 0.15)
 				)
 				(justify left bottom mirror)
-			)
-		)
-		(fp_text user "-"
-			(at -3 0.05 55)
-			(unlocked yes)
-			(layer "B.SilkS")
-			(effects
-				(font
-					(size 2 2)
-					(thickness 0.15)
-				)
-				(justify mirror)
 			)
 		)
@@
 		(embedded_fonts no)
 	)
-	(footprint "Alpenglow:LED_D5.0mm_Horizontal_O3.81mm_Z3.0mm_copy"
+	(footprint "Alpenglow:LED_D5.0mm_Horizontal"
 		(layer "B.Cu")
 		(at 146.587711 67.823037 155)
@@
 		(tags "LED")
 		(property "Reference" "D1"
-			(at 4.137566 -2.455649 335)
+			(at 4.089198 -2.322757 335)
 			(layer "B.SilkS")
 			(effects
@@
 			(layer "B.SilkS")
 			(hide yes)
+			(effects
+				(font
+					(size 1 1)
+					(thickness 0.15)
+				)
+				(justify mirror)
+			)
+		)
+		(property "Minus" "-"
+			(at 0 1.8 335)
+			(layer "B.SilkS")
+			(effects
+				(font
+					(size 1 1)
+					(thickness 0.15)
+				)
+				(justify mirror)
+			)
+		)
+		(property "Plus" "+"
+			(at 2.009821 1.736331 335)
+			(layer "B.SilkS")
 			(effects
 				(font
@@
 		)
 		(fp_line
-			(start -1.29 -3.75)
+			(start -1.29 -3.750001)
 			(end 3.83 -3.75)
 			(stroke
@@
 		)
 		(fp_line
-			(start -1.29 -3.75)
+			(start -1.29 -3.750001)
 			(end -1.29 -9.91)
 			(stroke
@@
 		(fp_arc
 			(start -1.29 -9.91)
-			(mid 1.27 -12.47)
+			(mid 1.27 -12.469999)
 			(end 3.83 -9.91)
 			(stroke
@@
 		(fp_poly
 			(pts
-				(xy -1.94 -12.719999) (xy 4.49 -12.72) (xy 4.49 1.21) (xy -1.94 1.21)
+				(xy -1.939999 -12.72) (xy 4.49 -12.72) (xy 4.49 1.21) (xy -1.94 1.21)
 			)
 			(stroke
@@
 			(fill no)
 			(layer "B.Fab")
-		)
-		(fp_text user "+"
-			(at 1.581095 1.053546 335)
-			(unlocked yes)
-			(layer "B.SilkS")
-			(effects
-				(font
-					(size 1 1)
-					(thickness 0.15)
-				)
-				(justify left bottom mirror)
-			)
-		)
-		(fp_text user "-"
-			(at -0.699999 1.2 335)
-			(unlocked yes)
-			(layer "B.SilkS")
-			(effects
-				(font
-					(size 1 1)
-					(thickness 0.15)
-				)
-				(justify left bottom mirror)
-			)
 		)
 		(fp_text user "${REFERENCE}"
@@
 		)
 	)
-	(footprint "Alpenglow:LED_D5.0mm_Horizontal_O3.81mm_Z3.0mm_copy"
+	(footprint "Alpenglow:LED_D5.0mm_Horizontal"
 		(layer "B.Cu")
 		(at 165.723375 66.74536 -155)
@@
 		(tags "LED")
 		(property "Reference" "D3"
-			(at 3.964365 -2.294173 25)
+			(at 4.284626 -2.034495 25)
 			(layer "B.SilkS")
 			(effects
@@
 			(layer "B.SilkS")
 			(hide yes)
+			(effects
+				(font
+					(size 1 1)
+					(thickness 0.15)
+				)
+				(justify mirror)
+			)
+		)
+		(property "Minus" "-"
+			(at -1.919065 0.148215 25)
+			(layer "B.SilkS")
+			(effects
+				(font
+					(size 1 1)
+					(thickness 0.15)
+				)
+				(justify mirror)
+			)
+		)
+		(property "Plus" "+"
+			(at 2.195475 1.735843 25)
+			(layer "B.SilkS")
 			(effects
 				(font
@@
 		(fp_arc
 			(start -1.29 -9.91)
-			(mid 1.270001 -12.469999)
+			(mid 1.27 -12.469998)
 			(end 3.83 -9.91)
 			(stroke
@@
 			(fill no)
 			(layer "B.Fab")
-		)
-		(fp_text user "+"
-			(at 1.85 1.2 25)
-			(unlocked yes)
-			(layer "B.SilkS")
-			(effects
-				(font
-					(size 1 1)
-					(thickness 0.15)
-				)
-				(justify left bottom mirror)
-			)
-		)
-		(fp_text user "-"
-			(at -0.7 1.2 25)
-			(unlocked yes)
-			(layer "B.SilkS")
-			(effects
-				(font
-					(size 1 1)
-					(thickness 0.15)
-				)
-				(justify left bottom mirror)
-			)
 		)
 		(fp_text user "${REFERENCE}"
@@
 		)
 	)
-	(footprint "Alpenglow:LED_D5.0mm_Horizontal_O3.81mm_Z3.0mm_copy"
+	(footprint "Alpenglow:LED_D5.0mm_Horizontal"
 		(layer "B.Cu")
 		(at 154.724999 134.155)
@@
 		(tags "LED")
 		(property "Reference" "D2"
-			(at 2.475001 2.445 180)
+			(at 2.575001 2.445 180)
 			(layer "B.SilkS")
 			(effects
@@
 			(layer "B.SilkS")
 			(hide yes)
+			(effects
+				(font
+					(size 1 1)
+					(thickness 0.15)
+				)
+				(justify mirror)
+			)
+		)
+		(property "Minus" "-"
+			(at -1.624999 -1.555 180)
+			(layer "B.SilkS")
+			(effects
+				(font
+					(size 1 1)
+					(thickness 0.15)
+				)
+				(justify mirror)
+			)
+		)
+		(property "Plus" "+"
+			(at 4.275001 0.045 180)
+			(layer "B.SilkS")
 			(effects
 				(font
@@
 		(duplicate_pad_numbers_are_jumpers no)
 		(fp_line
-			(start -1.29 -3.75)
+			(start -1.29 -3.750001)
 			(end -1.29 -9.91)
 			(stroke
@@
 		)
 		(fp_line
-			(start -1.29 -3.75)
+			(start -1.29 -3.750001)
 			(end 3.83 -3.75)
 			(stroke
@@
 			(layer "B.SilkS")
 		)
-		(fp_rect
-			(start 3.83 -3.75)
-			(end 4.23 -4.87)
-			(stroke
-				(width 0.12)
-				(type solid)
-			)
-			(fill no)
-			(layer "B.SilkS")
-		)
 		(fp_arc
 			(start -1.29 -9.91)
-			(mid 1.27 -12.47)
+			(mid 1.27 -12.469999)
 			(end 3.83 -9.91)
 			(stroke
@@
 			(layer "B.SilkS")
 		)
-		(fp_rect
-			(start -1.94 1.21)
-			(end 4.49 -12.72)
+		(fp_poly
+			(pts
+				(xy 3.83 -4.87) (xy 4.23 -4.87) (xy 4.229999 -3.75) (xy 3.83 -3.75)
+			)
+			(stroke
+				(width 0.12)
+				(type solid)
+			)
+			(fill no)
+			(layer "B.SilkS")
+		)
+		(fp_poly
+			(pts
+				(xy -1.939999 -12.72) (xy 4.49 -12.72) (xy 4.49 1.21) (xy -1.94 1.21)
+			)
 			(stroke
 				(width 0.05)
@@
 				(type solid)
 			)
-			(layer "B.Fab")
-		)
-		(fp_rect
-			(start 0 0)
-			(end 0 -3.81)
-			(stroke
-				(width 0.1)
-				(type solid)
-			)
-			(fill no)
-			(layer "B.Fab")
-		)
-		(fp_rect
-			(start 2.54 0)
-			(end 2.54 -3.81)
-			(stroke
-				(width 0.1)
-				(type solid)
-			)
-			(fill no)
-			(layer "B.Fab")
-		)
-		(fp_rect
-			(start 3.77 -3.81)
-			(end 4.17 -4.81)
-			(stroke
-				(width 0.1)
-				(type solid)
-			)
-			(fill no)
 			(layer "B.Fab")
 		)
@@
 			(layer "B.Fab")
 		)
-		(fp_text user "-"
-			(at -1.724999 -1.95 180)
-			(unlocked yes)
-			(layer "B.SilkS")
-			(effects
-				(font
-					(size 1 1)
-					(thickness 0.15)
-				)
-				(justify left bottom mirror)
-			)
-		)
-		(fp_text user "+"
-			(at 3.575001 -0.35 180)
-			(unlocked yes)
-			(layer "B.SilkS")
-			(effects
-				(font
-					(size 1 1)
-					(thickness 0.15)
-				)
-				(justify left bottom mirror)
-			)
+		(fp_poly
+			(pts
+				(xy 3.77 -4.81) (xy 4.17 -4.81) (xy 4.17 -3.81) (xy 3.77 -3.81)
+			)
+			(stroke
+				(width 0.1)
+				(type solid)
+			)
+			(fill no)
+			(layer "B.Fab")
 		)
 		(fp_text user "${REFERENCE}"

Commit message: Organized artwork into folder, linked all text to actual footprints in libraries
Parts:
- G2: renamed from ?; footprint clipboard:bf1500f7-63e0-4397-bbdb-e8a181ed9b95 -> FUterus:FUCK
- G3: renamed from ?; footprint clipboard:6fd78f95-30c4-45d5-b97f-0a242345d2c7 -> FUterus:OFF!
- G4: renamed from ?; footprint clipboard:9932db26-c585-4969-88a4-3276315666fc -> FUterus:aka the Boobterus
- G5: renamed from ?; footprint clipboard:978c0960-0638-40cb-9598-f7584c1d72e6 -> FUterus:The FUterus by Carrie Sundra
- renumbered G*** to G1
