File: Alpenglow_FUterus_PCB_test.kicad_pcb (KiCad board)
At the start: 2 copper layers, 76.2 x 76.2 mm, 12 parts, among them SW1 SW_SLIDE

Commit message: Cleaned up, added text, set components to DNP to avoid Fab Toolkit error, sent to JLC
Other:
- board text removed: "Destroy"
- board text removed: "Fascism"
